Commit message: Increase go2 joint torque/PID gains and swing height for climbing
- hip/thigh torque_max 23.7->45.0 Nm, calf 35.55->60.0 Nm
- joint PID: p 100->220, d 1.0->3.0, i_clamp 2.5->4.0
- gait swing_height 0.04->0.07m, stance_depth 0.01->0.02m
  (robot was unable to climb an incline with default gains)

File: go2_ws/src/unitree-go2-ros2/robots/descriptions/go2_description/xacro/const.xacro (robot description, xacro)
@@ -44,13 +44,13 @@
     <xacro:property name="hip_position_min" value="-1.0472"/>
     <xacro:property name="hip_velocity_max" value="30.1"/>
-    <xacro:property name="hip_torque_max" value="23.7"/>
+    <xacro:property name="hip_torque_max" value="45.0"/>
     <xacro:property name="thigh_position_max" value="3.4907"/>
     <xacro:property name="thigh_position_min" value="-1.5708"/>
     <xacro:property name="thigh_velocity_max" value="30.1"/>
-    <xacro:property name="thigh_torque_max" value="23.7"/>
+    <xacro:property name="thigh_torque_max" value="45.0"/>
     <xacro:property name="calf_position_max" value="-0.83776"/>
     <xacro:property name="calf_position_min" value="-2.7227"/>
     <xacro:property name="calf_velocity_max" value="20.06"/>
-    <xacro:property name="calf_torque_max" value="35.55"/>
+    <xacro:property name="calf_torque_max" value="60.0"/>
     <!-- dynamics inertial value -->
     <!-- trunk -->
